File: pcb/4-voice/1_1/4-voice(1_1).sch (EAGLE design)
At the start: 0 parts

Commit message: Add lots more parts, make sch of progress
Parts:
- added C1, C14, C16, C19, C20, C22, C23, C3, C5, C6: 0.1u, rcl:C-EUC1206
- added C10: 1u, rcl:C-EUC1206
- added C11, C12: 100n, rcl:C-EUC1206
- added C13: 4.7u, rcl:C-EUC1206
- added C15, C17, C18, C2: 10u, rcl:C-EUC1206
- added C21, C4: 22p, rcl:C-EUC1206
- added C24, C7: .001u, rcl:C-EUC1206
- added C25, C8: .002u, rcl:C-EUC1206
- added C9: 10n, rcl:C-EUC1206
- added JP1: (no value), pinhead:PINHD-1X6
- added R1, R2, R8, R9: 22k, rcl:R-US_R1206
- added R10, R3: 4.7k, rcl:R-US_R1206
- added R11, R4: 1k, rcl:R-US_R1206
- added R12, R13, R5, R6, R7: 10k, rcl:R-US_R1206
- added TP1, TP2: TPPAD1-13, testpad:TPPAD1-13
- added U$1, U$4: TL072, synth:TL072
- added U$2: STM32C8, synth:STM32C8
- added U$3: DAC084S085, synth:DAC084S085
- added U1, U2: THAT2180, synth:THAT2180
Connections:
- new net +15V: C19.2, C22.2, C3.2, C5.2, U$1G$3.V+, U$4G$3.V+, U1.V+, U2.V+
- new net +3V3: C10.1, C11.1, C12.1, C13.1, C14.1, C15.1, C16.1, C17.1, C9.1, JP1.5, U$2.VDD@1, U$2.VDD@2, U$2.VDDA, U$3.VA, U$3.V_REFIN
- new net -15V: C1.1, C20.1, C23.1, C24.1, C6.1, C7.1, U$1G$3.V-, U$4G$3.V-, U1.V-, U2.V-
- new net F-CTRL0: U$2.PA9
- new net F-CTRL1: U$2.PA0
- new net F-CTRL2: U$2.PA3
- new net F-CTRL3: U$2.PB0
- new net GND: C1.2, C10.2, C11.2, C12.2, C13.2, C14.2, C15.2, C16.2, C17.2, C19.1, C20.2, C22.1, C23.2, C3.1, C5.1, C6.2, C9.2, JP1.6, R11.1, R4.1, R7.2, U$1G$1.IN+, U$2.VSS@1, U$2.VSS@2, U$2.VSSA, U$3.GND, U$4G$1.IN+, U1.EC+, U1.GND, U2.EC+, U2.GND
- new net MOSI: U$2.PA7, U$3.DIN
- new net N$1: C2.2, R1.1
- new net N$10: R8.2, U2.-IN
- new net N$11: C21.1, R9.1, U$4G$1.IN-, U2.OUT
- new net N$12: R10.2, R11.2, R12.2
- new net N$13: C25.2, R12.1, R13.2
- new net N$14: C24.2, R13.1, U$4G$2.IN+
- new net N$2: R1.2, U1.-IN
- new net N$3: C4.1, R2.1, U$1G$1.IN-, U1.OUT
- new net N$4: R3.2, R4.2, R5.2
- new net N$5: C8.2, R5.1, R6.2
- new net N$6: C7.2, R6.1, U$1G$2.IN+
- new net N$7: TP1.TP, U$2.VBAT
- new net N$8: R7.1, TP2.TP, U$2.BOOT0
- new net N$9: C18.2, R8.1
- new net NRST: JP1.2, U$2.NRST
- new net NSS: U$2.PA4, U$3.!SYNC
- new net OSC1: C2.1, U$3.V_OUTA
- new net OSC2: C18.1, U$3.V_OUTB
- new net OSC3: U$3.V_OUTC
- new net OSC4: U$3.V_OUTD
- new net Q-CTRL0: U$2.PA10
- new net Q-CTRL1: U$2.PA1
- new net Q-CTRL2: U$2.PB4
- new net Q-CTRL3: U$2.PB1
- new net SCK: U$2.PA5, U$3.SCLK
- new net SWCLK: JP1.3, U$2.PA14
- new net SWDIO: JP1.4, U$2.PA13
- new net SWO: JP1.1, U$2.PB3
- new net VCA-CTRL0: R3.1, U$2.PA8
- new net VCA-CTRL1: R10.1, U$2.PA11
- new net VCA-CTRL2: U$2.PA2
- new net VCA-CTRL3: U$2.PB5
- new net VCA0: C8.1, U$1G$2.IN-, U$1G$2.OUT, U1.EC-
- new net VCA1: C25.1, U$4G$2.IN-, U$4G$2.OUT, U2.EC-
- new net VCA_OUT1: C4.2, R2.2, U$1G$1.OUT
- new net VCA_OUT2: C21.2, R9.2, U$4G$1.OUT
Other:
- note added: "VDD VSS"
- note added: "VDDA VSSA"
