File: pcb/4-voice/1_1/4-voice(1_1).sch (EAGLE design)
At the start: 47 parts, among them U1 THAT2180, U2 THAT2180

Commit message: Add filter, start lin-expo converter
Parts:
- added C26, C34: 10u, rcl:C-EUC1206
- added C27, C28, C30, C31, C35, C36, C38, C39: 0.1u, rcl:C-EUC1206
- added C29, C37: 22p, rcl:C-EUC1206
- added C32, C40: .001u, rcl:C-EUC1206
- added C33, C41: .002u, rcl:C-EUC1206
- added C42: 1000p, resistor:C-EUC1206
- added C43: 2000p, resistor:C-EUC1206
- added C44, C45: 0.1u, resistor:C-EUC1206
- added C46: 1n, resistor:C-EUC1206
- added R14, R15, R20, R21: 22k, rcl:R-US_R1206
- added R16, R22: 4.7k, rcl:R-US_R1206
- added R17, R23: 1k, rcl:R-US_R1206
- added R18, R19, R24, R25: 10k, rcl:R-US_R1206
- added R26, R33, R35, R37: 100k, resistor:R-US_R1206
- added R27, R30, R32, R34: 2k, resistor:R-US_R1206
- added R28: 15k, resistor:R-US_R1206
- added R29: 100K, resistor:R-US_R1206
- added R31, R36: 10k, resistor:R-US_R1206
- added R38: 1.8k, resistor:R-US_R1206
- added R39: 1k, resistor:R-US_R1206
- added U$10: (no value), LITTLEBITS:XX-13700DMP16
- added U$11, U$5, U$6, U$7, U$8, U$9: TL072, synth:TL072
- added U3, U4: THAT2180, synth:THAT2180
- U$4: SPICEPREFIX (none) -> J
Connections:
- removed net OSC4: U$3.V_OUTD
- new net FILT_IN: R26.1
- new net FILT_OUT: C42.2, R35.1, R36.1, U$10G$2.BUFF/OUT
- new net F_IN: R28.2
- new net N$15: C26.2, R14.1
- new net N$16: R14.2, U3.-IN
- new net N$17: C29.1, R15.1, U$5G$1.IN-, U3.OUT
- new net N$18: R16.2, R17.2, R18.2
- new net N$19: C33.2, R18.1, R19.2
- new net N$20: C32.2, R19.1, U$6G$2.IN+
- new net N$21: C34.2, R20.1
- new net N$22: R20.2, U4.-IN
- new net N$23: C37.1, R21.1, U$7G$1.IN-, U4.OUT
- new net N$24: R22.2, R23.2, R24.2
- new net N$25: C41.2, R24.1, R25.2
- new net N$26: C40.2, R25.1, U$9G$2.IN+
- new net N$27: R26.2, R27.2, U$10G$1.+IN
- new net N$28: R28.1, U$10G$1.AMP/BIAS, U$10G$2.AMP/BIAS
- new net N$29: R37.1, R38.2, U$11G$1.IN-
- new net N$30: R37.2
- new net N$31: R29.2, R30.1, U$10G$1.-IN
- new net N$32: C42.1, U$10G$1.BUFF/IN, U$10G$1.OUT
- new net N$33: R29.1, R31.1, R33.1, U$10G$1.BUFF/OUT
- new net N$34: C43.1, U$10G$2.BUFF/IN, U$10G$2.OUT
- new net N$35: R32.1, R33.2, U$10G$2.+IN
- new net N$36: R34.1, R35.2, U$10G$2.-IN
- new net N$37: R38.1, U$11G$1.OUT
- new net N$38: C46.2, R39.1, U$11G$2.OUT
- new net N$39: C46.1, U$11G$2.IN-
- new net OSC0: C2.1, U$3.V_OUTA
- new net VCA2: C33.1, U$6G$2.IN-, U$6G$2.OUT, U3.EC-
- new net VCA3: C41.1, U$9G$2.IN-, U$9G$2.OUT, U4.EC-
- new net VCA_OUT0: C4.2, R2.2, U$1G$1.OUT
- new net VCA_OUT3: C37.2, R21.2, U$7G$1.OUT
- net +15V: now also C27.2, C30.2, C35.2, C38.2, C44.1, U$10G$3.VCC, U$6G$3.V+, U$8G$3.V+, U3.V+, U4.V+
- net -15V: now also C28.1, C31.1, C32.1, C36.1, C39.1, C40.1, C45.2, R31.2, R36.2, U$10G$3.GND, U$6G$3.V-, U$8G$3.V-, U3.V-, U4.V-
- net GND: now also C27.1, C28.2, C30.1, C31.2, C35.1, C36.2, C38.1, C39.2, C43.2, C44.2, C45.1, R17.1, R23.1, R27.1, R30.2, R32.2, R34.2, U$11G$1.IN+, U$11G$2.IN+, U$5G$1.IN+, U$7G$1.IN+, U3.EC+, U3.GND, U4.EC+, U4.GND
- net OSC1: now also C18.1, U$3.V_OUTB; no longer C2.1, U$3.V_OUTA
- net OSC2: now also C26.1, U$3.V_OUTC; no longer C18.1, U$3.V_OUTB
- net OSC3: now also C34.1, U$3.V_OUTD; no longer U$3.V_OUTC
- net VCA-CTRL2: now also R16.1
- net VCA-CTRL3: now also R22.1
- net VCA_OUT1: now also C21.2, R9.2, U$4G$1.OUT; no longer C4.2, R2.2, U$1G$1.OUT
- net VCA_OUT2: now also C29.2, R15.2, U$5G$1.OUT; no longer C21.2, R9.2, U$4G$1.OUT
