File: pcb/4-voice/1_1/4-voice(1_1).brd (EAGLE design)
At the start: 160 x 100 mm, 0 parts

Commit message: Add lots more parts, make sch of progress
Parts:
- added C1, C14, C16, C19, C20, C22, C23, C3, C5, C6: 0.1u, rcl:C1206
- added C10: 1u, rcl:C1206
- added C11, C12: 100n, rcl:C1206
- added C13: 4.7u, rcl:C1206
- added C15, C17, C18, C2: 10u, rcl:C1206
- added C21, C4: 22p, rcl:C1206
- added C24, C7: .001u, rcl:C1206
- added C25, C8: .002u, rcl:C1206
- added C9: 10n, rcl:C1206
- added JP1: (no value), pinhead:1X06
- added R1, R2, R8, R9: 22k, rcl:R1206
- added R10, R3: 4.7k, rcl:R1206
- added R11, R4: 1k, rcl:R1206
- added R12, R13, R5, R6, R7: 10k, rcl:R1206
- added TP1, TP2: TPPAD1-13, testpad:P1-13
- added U$1, U$4: TL072, synth:SOIC8
- added U$2: STM32C8, synth:LQFP48
- added U$3: DAC084S085, synth:VSSOP10
- added U1, U2: THAT2180, synth:SIP8
Connections:
- new net +15V: C19.2, C22.2, C3.2, C5.2, U$1.P$8, U$4.P$8, U1.$P7, U2.$P7
- new net +3V3: C10.1, C11.1, C12.1, C13.1, C14.1, C15.1, C16.1, C17.1, C9.1, JP1.5, U$2.P$24, U$2.P$48, U$2.P$9, U$3.P$1, U$3.P$7
- new net -15V: C1.1, C20.1, C23.1, C24.1, C6.1, C7.1, U$1.P$4, U$4.P$4, U1.$P5, U2.$P5
- new net F-CTRL0: U$2.P$30
- new net F-CTRL1: U$2.P$10
- new net F-CTRL2: U$2.P$13
- new net F-CTRL3: U$2.P$18
- new net GND: C1.2, C10.2, C11.2, C12.2, C13.2, C14.2, C15.2, C16.2, C17.2, C19.1, C20.2, C22.1, C23.2, C3.1, C5.1, C6.2, C9.2, JP1.6, R11.1, R4.1, R7.2, U$1.P$3, U$2.P$23, U$2.P$47, U$2.P$8, U$3.P$6, U$4.P$3, U1.$P2, U1.$P6, U2.$P2, U2.$P6
- new net MOSI: U$2.P$17, U$3.P$8
- new net N$1: C2.2, R1.1
- new net N$10: R8.2, U2.$P1
- new net N$11: C21.1, R9.1, U$4.P$2, U2.$P8
- new net N$12: R10.2, R11.2, R12.2
- new net N$13: C25.2, R12.1, R13.2
- new net N$14: C24.2, R13.1, U$4.P$5
- new net N$2: R1.2, U1.$P1
- new net N$3: C4.1, R2.1, U$1.P$2, U1.$P8
- new net N$4: R3.2, R4.2, R5.2
- new net N$5: C8.2, R5.1, R6.2
- new net N$6: C7.2, R6.1, U$1.P$5
- new net N$7: TP1.TP, U$2.P$1
- new net N$8: R7.1, TP2.TP, U$2.P$44
- new net N$9: C18.2, R8.1
- new net NRST: JP1.2, U$2.P$7
- new net NSS: U$2.P$14, U$3.P$9
- new net OSC1: C2.1, U$3.P$2
- new net OSC2: C18.1, U$3.P$3
- new net OSC3: U$3.P$4
- new net OSC4: U$3.P$5
- new net Q-CTRL0: U$2.P$31
- new net Q-CTRL1: U$2.P$11
- new net Q-CTRL2: U$2.P$40
- new net Q-CTRL3: U$2.P$19
- new net SCK: U$2.P$15, U$3.P$10
- new net SWCLK: JP1.3, U$2.P$37
- new net SWDIO: JP1.4, U$2.P$34
- new net SWO: JP1.1, U$2.P$39
- new net VCA-CTRL0: R3.1, U$2.P$29
- new net VCA-CTRL1: R10.1, U$2.P$32
- new net VCA-CTRL2: U$2.P$12
- new net VCA-CTRL3: U$2.P$41
- new net VCA0: C8.1, U$1.P$6, U$1.P$7, U1.$P3
- new net VCA1: C25.1, U$4.P$6, U$4.P$7, U2.$P3
- new net VCA_OUT1: C4.2, R2.2, U$1.P$1
- new net VCA_OUT2: C21.2, R9.2, U$4.P$1

Commit message: Add filter, start lin-expo converter
Parts:
- added C26, C34: 10u, rcl:C1206
- added C27, C28, C30, C31, C35, C36, C38, C39: 0.1u, rcl:C1206
- added C29, C37: 22p, rcl:C1206
- added C32, C40: .001u, rcl:C1206
- added C33, C41: .002u, rcl:C1206
- added C42: 1000p, resistor:C1206
- added C43: 2000p, resistor:C1206
- added C44, C45: 0.1u, resistor:C1206
- added C46: 1n, resistor:C1206
- added R14, R15, R20, R21: 22k, rcl:R1206
- added R16, R22: 4.7k, rcl:R1206
- added R17, R23: 1k, rcl:R1206
- added R18, R19, R24, R25: 10k, rcl:R1206
- added R26, R33, R35, R37: 100k, resistor:R1206
- added R27, R30, R32, R34: 2k, resistor:R1206
- added R28: 15k, resistor:R1206
- added R29: 100K, resistor:R1206
- added R31, R36: 10k, resistor:R1206
- added R38: 1.8k, resistor:R1206
- added R39: 1k, resistor:R1206
- added U$10: (no value), LITTLEBITS:DMP16
- added U$11, U$5, U$6, U$7, U$8, U$9: TL072, synth:SOIC8
- added U3, U4: THAT2180, synth:SIP8
Connections:
- removed net OSC4: U$3.P$5
- new net FILT_IN: R26.1
- new net FILT_OUT: C42.2, R35.1, R36.1, U$10.9
- new net F_IN: R28.2
- new net N$15: C26.2, R14.1
- new net N$16: R14.2, U3.$P1
- new net N$17: C29.1, R15.1, U$5.P$2, U3.$P8
- new net N$18: R16.2, R17.2, R18.2
- new net N$19: C33.2, R18.1, R19.2
- new net N$20: C32.2, R19.1, U$6.P$5
- new net N$21: C34.2, R20.1
- new net N$22: R20.2, U4.$P1
- new net N$23: C37.1, R21.1, U$7.P$2, U4.$P8
- new net N$24: R22.2, R23.2, R24.2
- new net N$25: C41.2, R24.1, R25.2
- new net N$26: C40.2, R25.1, U$9.P$5
- new net N$27: R26.2, R27.2, U$10.3
- new net N$28: R28.1, U$10.1, U$10.16
- new net N$29: R37.1, R38.2, U$11.P$2
- new net N$30: R37.2
- new net N$31: R29.2, R30.1, U$10.4
- new net N$32: C42.1, U$10.5, U$10.7
- new net N$33: R29.1, R31.1, R33.1, U$10.8
- new net N$34: C43.1, U$10.10, U$10.12
- new net N$35: R32.1, R33.2, U$10.14
- new net N$36: R34.1, R35.2, U$10.13
- new net N$37: R38.1, U$11.P$1
- new net N$38: C46.2, R39.1, U$11.P$7
- new net N$39: C46.1, U$11.P$6
- new net OSC0: C2.1, U$3.P$2
- new net VCA2: C33.1, U$6.P$6, U$6.P$7, U3.$P3
- new net VCA3: C41.1, U$9.P$6, U$9.P$7, U4.$P3
- new net VCA_OUT0: C4.2, R2.2, U$1.P$1
- new net VCA_OUT3: C37.2, R21.2, U$7.P$1
- net +15V: now also C27.2, C30.2, C35.2, C38.2, C44.1, U$10.11, U$6.P$8, U$8.P$8, U3.$P7, U4.$P7
- net -15V: now also C28.1, C31.1, C32.1, C36.1, C39.1, C40.1, C45.2, R31.2, R36.2, U$10.6, U$6.P$4, U$8.P$4, U3.$P5, U4.$P5
- net GND: now also C27.1, C28.2, C30.1, C31.2, C35.1, C36.2, C38.1, C39.2, C43.2, C44.2, C45.1, R17.1, R23.1, R27.1, R30.2, R32.2, R34.2, U$11.P$3, U$11.P$5, U$5.P$3, U$7.P$3, U3.$P2, U3.$P6, U4.$P2, U4.$P6
- net OSC1: now also C18.1, U$3.P$3; no longer C2.1, U$3.P$2
- net OSC2: now also C26.1, U$3.P$4; no longer C18.1, U$3.P$3
- net OSC3: now also C34.1, U$3.P$5; no longer U$3.P$4
- net VCA-CTRL2: now also R16.1
- net VCA-CTRL3: now also R22.1
- net VCA_OUT1: now also C21.2, R9.2, U$4.P$1; no longer C4.2, R2.2, U$1.P$1
- net VCA_OUT2: now also C29.2, R15.2, U$5.P$1; no longer C21.2, R9.2, U$4.P$1
