File: pcb/1-voice/1_1/1-voice(1_1).brd (EAGLE design)
At the start: 160 x 100 mm, 103 parts, among them U1 THAT2180, U2 THAT2180, U3 THAT2180, U4 THAT2180

Commit message: move 4voice to 1voice, do lin->exp
Parts:
- removed C21, C29, C37: 22p, rcl:C1206
- removed C22, C23, C27, C28, C30, C31, C35, C36, C38, C39: 0.1u, rcl:C1206
- removed C24, C32, C40: .001u, rcl:C1206
- removed C25, C33, C41: .002u, rcl:C1206
- removed C26, C34: 10u, rcl:C1206
- removed C46: 1n, resistor:C1206
- removed R10, R16, R22: 4.7k, rcl:R1206
- removed R11, R17, R23: 1k, rcl:R1206
- removed R12, R13, R18, R19, R24, R25: 10k, rcl:R1206
- removed R14, R15, R20, R21: 22k, rcl:R1206
- removed R37: 100k, resistor:R1206
- removed R38: 1.8k, resistor:R1206
- removed R39: 1k, resistor:R1206
- removed U$4, U$5, U$6, U$7, U$8, U$9: TL072, synth:SOIC8
- removed U2, U3, U4: THAT2180, synth:SIP8
- added Q1, Q2: (no value), LITTLEBITS:SOT-363-JBLMASK
- C18: value 10u -> 0.1u
- C20: value 0.1u -> 10u
- R8: value 22k -> 1k; device rcl:R1206 -> resistor:R1206
- R9: value 22k -> 2.7M; device rcl:R1206 -> resistor:R1206
- moved C20 395.7 mm to (-63.5, -603.2)
- moved C19 393.6 mm to (-57.1, -590.5)
- moved R9 389.4 mm to (-63.5, -609.6)
- moved R8 385.6 mm to (-63.5, -596.9)
- moved C18 370.5 mm to (-57.1, -584.2)
Connections:
- removed net N$12: R10.2, R11.2, R12.2
- removed net N$14: C24.2, R13.1, U$4.P$5
- removed net N$15: C26.2, R14.1
- removed net N$16: R14.2, U3.$P1
- removed net N$17: C29.1, R15.1, U$5.P$2, U3.$P8
- removed net N$18: R16.2, R17.2, R18.2
- removed net N$19: C33.2, R18.1, R19.2
- removed net N$20: C32.2, R19.1, U$6.P$5
- removed net N$21: C34.2, R20.1
- removed net N$22: R20.2, U4.$P1
- removed net N$23: C37.1, R21.1, U$7.P$2, U4.$P8
- removed net N$24: R22.2, R23.2, R24.2
- removed net N$25: C41.2, R24.1, R25.2
- removed net N$26: C40.2, R25.1, U$9.P$5
- removed net N$29: R37.1, R38.2, U$11.P$2
- removed net N$30: R37.2
- removed net N$37: R38.1, U$11.P$1
- removed net N$38: C46.2, R39.1, U$11.P$7
- removed net N$39: C46.1, U$11.P$6
- removed net VCA1: C25.1, U$4.P$6, U$4.P$7, U2.$P3
- removed net VCA2: C33.1, U$6.P$6, U$6.P$7, U3.$P3
- removed net VCA3: C41.1, U$9.P$6, U$9.P$7, U4.$P3
- removed net VCA_OUT1: C21.2, R9.2, U$4.P$1
- removed net VCA_OUT2: C29.2, R15.2, U$5.P$1
- removed net VCA_OUT3: C37.2, R21.2, U$7.P$1
- new net F_LIN: Q1.2
- net +15V: now also C18.2, Q2.1, Q2.4, R9.2, U$11.P$8; no longer C19.2, C22.2, C27.2, C30.2, C35.2, C38.2, U$4.P$8, U$6.P$8, U$8.P$8, U2.$P7, U3.$P7, U4.$P7
- net -15V: now also C19.1, U$11.P$4; no longer C20.1, C23.1, C24.1, C28.1, C31.1, C32.1, C36.1, C39.1, C40.1, U$4.P$4, U$6.P$4, U$8.P$4, U2.$P5, U3.$P5, U4.$P5
- net F_IN: now also Q2.6
- net GND: now also C18.1, C19.2, Q1.5; no longer C19.1, C20.2, C22.1, C23.2, C27.1, C28.2, C30.1, C31.2, C35.1, C36.2, C38.1, C39.2, R11.1, R17.1, R23.1, U$11.P$5, U$4.P$3, U$5.P$3, U$7.P$3, U2.$P2, U2.$P6, U3.$P2, U3.$P6, U4.$P2, U4.$P6
- net N$10: now also C20.2, R8.1, U$11.P$1; no longer R8.2, U2.$P1
- net N$11: now also C20.1, Q1.6, U$11.P$2; no longer C21.1, U$4.P$2, U2.$P8
- net N$13: now also Q1.3, Q2.2, Q2.3, Q2.5; no longer C25.2, R12.1, R13.2
- net N$9: now also Q1.1, Q1.4, R8.2; no longer C18.2, R8.1
- net OSC1: no longer C18.1
- net OSC2: no longer C26.1
- net OSC3: no longer C34.1
- net VCA-CTRL1: no longer R10.1
- net VCA-CTRL2: no longer R16.1
- net VCA-CTRL3: no longer R22.1
