File: pcb/1-voice/1_1/1-voice(1_1).sch (EAGLE design)
At the start: 103 parts, among them U1 THAT2180, U2 THAT2180, U3 THAT2180, U4 THAT2180

Commit message: move 4voice to 1voice, do lin->exp
Parts:
- removed C21, C29, C37: 22p, rcl:C-EUC1206
- removed C22, C23, C27, C28, C30, C31, C35, C36, C38, C39: 0.1u, rcl:C-EUC1206
- removed C24, C32, C40: .001u, rcl:C-EUC1206
- removed C25, C33, C41: .002u, rcl:C-EUC1206
- removed C26, C34: 10u, rcl:C-EUC1206
- removed C46: 1n, resistor:C-EUC1206
- removed R10, R16, R22: 4.7k, rcl:R-US_R1206
- removed R11, R17, R23: 1k, rcl:R-US_R1206
- removed R12, R13, R18, R19, R24, R25: 10k, rcl:R-US_R1206
- removed R14, R15, R20, R21: 22k, rcl:R-US_R1206
- removed R37: 100k, resistor:R-US_R1206
- removed R38: 1.8k, resistor:R-US_R1206
- removed R39: 1k, resistor:R-US_R1206
- removed U$4, U$5, U$6, U$7, U$8, U$9: TL072, synth:TL072
- removed U2, U3, U4: THAT2180, synth:THAT2180
- added Q1: (no value), LITTLEBITS:TRANS-BJT_NPN-DUAL-BC847BS-JBLMASK
- added Q2: (no value), LITTLEBITS:TRANS-BJT_PNP-DUAL-BC857-JBLMASK
- C18: value 10u -> 0.1u
- C20: value 0.1u -> 10u
- R8: value 22k -> 1k; device rcl:R-US_R1206 -> resistor:R-US_R1206
- R9: value 22k -> 2.7M; device rcl:R-US_R1206 -> resistor:R-US_R1206
Connections:
- removed net N$12: R10.2, R11.2, R12.2
- removed net N$14: C24.2, R13.1, U$4G$2.IN+
- removed net N$15: C26.2, R14.1
- removed net N$16: R14.2, U3.-IN
- removed net N$17: C29.1, R15.1, U$5G$1.IN-, U3.OUT
- removed net N$18: R16.2, R17.2, R18.2
- removed net N$19: C33.2, R18.1, R19.2
- removed net N$20: C32.2, R19.1, U$6G$2.IN+
- removed net N$21: C34.2, R20.1
- removed net N$22: R20.2, U4.-IN
- removed net N$23: C37.1, R21.1, U$7G$1.IN-, U4.OUT
- removed net N$24: R22.2, R23.2, R24.2
- removed net N$25: C41.2, R24.1, R25.2
- removed net N$26: C40.2, R25.1, U$9G$2.IN+
- removed net N$29: R37.1, R38.2, U$11G$1.IN-
- removed net N$30: R37.2
- removed net N$37: R38.1, U$11G$1.OUT
- removed net N$38: C46.2, R39.1, U$11G$2.OUT
- removed net N$39: C46.1, U$11G$2.IN-
- removed net VCA1: C25.1, U$4G$2.IN-, U$4G$2.OUT, U2.EC-
- removed net VCA2: C33.1, U$6G$2.IN-, U$6G$2.OUT, U3.EC-
- removed net VCA3: C41.1, U$9G$2.IN-, U$9G$2.OUT, U4.EC-
- removed net VCA_OUT1: C21.2, R9.2, U$4G$1.OUT
- removed net VCA_OUT2: C29.2, R15.2, U$5G$1.OUT
- removed net VCA_OUT3: C37.2, R21.2, U$7G$1.OUT
- new net F_LIN: Q1A.B
- net +15V: now also C18.2, Q2A.E, Q2B.E, R9.2, U$11G$3.V+; no longer C19.2, C22.2, C27.2, C30.2, C35.2, C38.2, U$4G$3.V+, U$6G$3.V+, U$8G$3.V+, U2.V+, U3.V+, U4.V+
- net -15V: now also C19.1, U$11G$3.V-; no longer C20.1, C23.1, C24.1, C28.1, C31.1, C32.1, C36.1, C39.1, C40.1, U$4G$3.V-, U$6G$3.V-, U$8G$3.V-, U2.V-, U3.V-, U4.V-
- net F_IN: now also Q2A.C
- net GND: now also C18.1, C19.2, Q1B.B; no longer C19.1, C20.2, C22.1, C23.2, C27.1, C28.2, C30.1, C31.2, C35.1, C36.2, C38.1, C39.2, R11.1, R17.1, R23.1, U$11G$2.IN+, U$4G$1.IN+, U$5G$1.IN+, U$7G$1.IN+, U2.EC+, U2.GND, U3.EC+, U3.GND, U4.EC+, U4.GND
- net N$10: now also C20.2, R8.1, U$11G$1.OUT; no longer R8.2, U2.-IN
- net N$11: now also C20.1, Q1A.C, U$11G$1.IN-; no longer C21.1, U$4G$1.IN-, U2.OUT
- net N$13: now also Q1B.C, Q2A.B, Q2B.B, Q2B.C; no longer C25.2, R12.1, R13.2
- net N$9: now also Q1A.E, Q1B.E, R8.2; no longer C18.2, R8.1
- net OSC1: no longer C18.1
- net OSC2: no longer C26.1
- net OSC3: no longer C34.1
- net VCA-CTRL1: no longer R10.1
- net VCA-CTRL2: no longer R16.1
- net VCA-CTRL3: no longer R22.1
