File: pcb/1-voice/2_2/1-voice(2_2).brd (EAGLE design)
At the start: 75 x 30 mm, 74 parts, among them U1 THAT2180

Commit message: Made v2
Parts:
- removed TP1: TPB1,27, testpad:B1,27
- added C26: 0.1u, rcl:C0603
- added LED1, LED2, LED3, LED4: (no value), led:1206
- added R14: 5.1k, rcl:R0603
- added R15: 20k, rcl:R0603
- added R16: 330k, rcl:R0603
- added R17, R18: 4.7k, rcl:R0603
- added R19, R20, R21, R22: 1k, rcl:R0603
- added SJ1: (no value), jumper:SJ
- added U$5: TL072, synth:SOIC8
- added U$6: SWITCH-DPDT, synth:DPDT
- C25: value 10u -> 0.1u
- R10: value 4.7k -> 20k
- R13: value 330 -> 330k
- moved JP1 15.6 mm to (10.8, 2.10), turned to 0 degrees
- moved C21 13.1 mm to (14.2, 27.1), turned to 180 degrees
- moved U$4 11.1 mm to (13.9, 24.5), turned to 90 degrees
- moved C25 9.73 mm to (34.9, 13.8), turned to 90 degrees
- moved R13 8.72 mm to (35.4, 19.0), turned to 270 degrees
- moved C22 8.64 mm to (15.3, 21.6), turned to 0 degrees
- moved JP10 6.10 mm to (31.3, 5.90)
- moved JP11 6.10 mm to (31.3, 17.0)
- moved R10 5.80 mm to (37.5, 19.0), turned to 90 degrees
- moved TP3 5.47 mm to (19.5, 20.9)
- moved JP8 5.40 mm to (27.7, 5.90)
- moved JP9 5.40 mm to (27.7, 17.0)
- moved C10 4.81 mm to (10.3, 6.40)
- moved C14 4.80 mm to (20.4, 15.2)
- moved C15 4.80 mm to (20.4, 17.2)
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Connections:
- new net -15V-IN: JP7.1, U$6.P$5
- new net 15V-IN: JP7.3, U$6.P$2
- new net LED: LED4.A, U$2.P$38
- new net N$16: R14.2, U1.$P5
- new net N$17: LED1.C, R19.2
- new net N$18: LED2.C, R20.2
- new net N$19: R16.1, R17.2, R18.1
- new net N$20: R15.1, R16.2, U$5.P$5
- new net N$21: LED3.A, R21.2
- new net N$22: LED4.C, R22.2
- net +15V: now also C25.2, LED1.A, U$5.P$8, U$6.P$1; no longer JP7.3
- net +3V3: now also LED2.A, R18.2
- net -15V: now also C26.1, LED3.C, R14.1, U$5.P$4, U$6.P$4; no longer JP7.1, U1.$P5
- net F-CTRL0: now also R13.2; no longer C25.1
- net F-CTRL0-EXP: now also SJ1.1; no longer Q2.6
- net GND: now also C25.1, C26.2, R15.2, R17.1, R19.1, R20.1, R21.1, R22.1; no longer R13.1
- net N$1: now also R10.2, R13.1, U$5.P$6; no longer C25.2, R10.1
- net N$15: now also R10.1, U$5.P$7; no longer R10.2, R13.2
- net N$7: now also Q2.6, SJ1.2; no longer TP1.TP, U$2.P$1
Routing:
- net -15V: track 120.4 -> 164.7 mm, vias 7 -> 9
- net +15V: track 104.2 -> 139.7 mm, vias 6 -> 10
- net +3V3: track 85.8 -> 104.0 mm
- net -15V-IN: track 0.00 -> 16.9 mm
- net LED: track 0.00 -> 14.0 mm, vias 0 -> 2
- net N$15: track 7.60 -> 19.1 mm, vias 0 -> 2
- net 15V-IN: track 0.00 -> 10.6 mm
- net OSC0-OUT: track 16.7 -> 25.4 mm
- net SWCLK: track 9.31 -> 17.3 mm, vias 0 -> 2
- net SWDIO: track 11.8 -> 18.6 mm, vias 0 -> 2
- net NRST: track 15.0 -> 9.20 mm, vias 1 -> 0
- net F-CTRL0: track 51.7 -> 47.0 mm
- net N$20: track 0.00 -> 4.12 mm
- net N$1: track 2.80 -> 6.17 mm
- net N$19: track 0.00 -> 3.29 mm
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Other:
- board size 75 x 30 mm -> 72.6 x 30 mm
- board text added: "190521"
- board text removed: "190507"

Commit message: Add LED blink code, Update schem with LED R values
Parts:
- R19: value 1k -> 100k
- R21: value 1k -> 10k
Changed lines of the file:
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@@
 <?xml version="1.0" encoding="utf-8"?>
 <!DOCTYPE eagle SYSTEM "eagle.dtd">
-<eagle version="9.2.1">
+<eagle version="9.3.2">
 <drawing>
 <settings>
@@
 <attribute name="VALUE" x="10.94" y="25.63" size="1.27" layer="27" rot="R90"/>
 </element>
-<element name="R19" library="rcl" library_urn="urn:adsk.eagle:library:334" package="R0603" package3d_urn="urn:adsk.eagle:package:23555/3" value="1k" x="10.6" y="22.9" smashed="yes" rot="R90">
+<element name="R19" library="rcl" library_urn="urn:adsk.eagle:library:334" package="R0603" package3d_urn="urn:adsk.eagle:package:23555/3" value="100k" x="10.6" y="22.9" smashed="yes" rot="R90">
 <attribute name="SPICEPREFIX" value="R" x="10.6" y="22.9" size="1.778" layer="27" rot="R90" display="off"/>
 </element>
@@
 <attribute name="SPICEPREFIX" value="R" x="6.2" y="22.9" size="1.778" layer="27" rot="R90" display="off"/>
 </element>
-<element name="R21" library="rcl" library_urn="urn:adsk.eagle:library:334" package="R0603" package3d_urn="urn:adsk.eagle:package:23555/3" value="1k" x="8.4" y="22.9" smashed="yes" rot="R90">
+<element name="R21" library="rcl" library_urn="urn:adsk.eagle:library:334" package="R0603" package3d_urn="urn:adsk.eagle:package:23555/3" value="10k" x="8.4" y="22.9" smashed="yes" rot="R90">
 <attribute name="SPICEPREFIX" value="R" x="8.4" y="22.9" size="1.778" layer="27" rot="R90" display="off"/>
 </element>

Commit message: Found error in sch values around lin->exp converter
Parts:
- Q1: value (none) -> NPN
- Q2: value (none) -> PNP
Changed lines of the file:
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@@
 <attribute name="SPICEPREFIX" value="C" x="45.7" y="7.5" size="1.778" layer="27" rot="R180" display="off"/>
 </element>
-<element name="Q1" library="LITTLEBITS" package="SOT-363-JBLMASK" value="" x="54.05" y="18.66" smashed="yes" rot="R270">
+<element name="Q1" library="LITTLEBITS" package="SOT-363-JBLMASK" value="NPN" x="54.05" y="18.66" smashed="yes" rot="R270">
 <attribute name="VALUE" x="51.985" y="19.76" size="0.4064" layer="27" font="vector" rot="R270"/>
 </element>
-<element name="Q2" library="LITTLEBITS" package="SOT-363-JBLMASK" value="" x="50.85" y="18.67" smashed="yes" rot="R270">
+<element name="Q2" library="LITTLEBITS" package="SOT-363-JBLMASK" value="PNP" x="50.85" y="18.67" smashed="yes" rot="R270">
 <attribute name="VALUE" x="48.785" y="19.77" size="0.4064" layer="27" font="vector" rot="R270"/>
 </element>
