File: pcb/1-voice/3_3/1-voice(3_3).sch (EAGLE design)
At the start: 90 parts, among them U1 THAT2180

Commit message: Add LED blink code, Update schem with LED R values
Parts:
- LED1: value (none) -> BLUE
- LED2: value (none) -> RED
- LED3: value (none) -> YELLOW
- LED4: value (none) -> GREEN
- R19: value 1k -> 100k
- R21: value 1k -> 10k
- R22: value 1k -> 470R
Changed lines of the file:
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@@
 <?xml version="1.0" encoding="utf-8"?>
 <!DOCTYPE eagle SYSTEM "eagle.dtd">
-<eagle version="9.2.1">
+<eagle version="9.3.2">
 <drawing>
 <settings>
@@
 <part name="C26" library="rcl" library_urn="urn:adsk.eagle:library:334" deviceset="C-EU" device="C0603" package3d_urn="urn:adsk.eagle:package:23616/2" value="0.1u"/>
 <part name="GND21" library="supply1" library_urn="urn:adsk.eagle:library:371" deviceset="GND" device=""/>
-<part name="LED1" library="led" library_urn="urn:adsk.eagle:library:259" deviceset="LED" device="SMT1206" package3d_urn="urn:adsk.eagle:package:15796/2"/>
-<part name="LED2" library="led" library_urn="urn:adsk.eagle:library:259" deviceset="LED" device="SMT1206" package3d_urn="urn:adsk.eagle:package:15796/2"/>
-<part name="LED3" library="led" library_urn="urn:adsk.eagle:library:259" deviceset="LED" device="SMT1206" package3d_urn="urn:adsk.eagle:package:15796/2"/>
+<part name="LED1" library="led" library_urn="urn:adsk.eagle:library:259" deviceset="LED" device="SMT1206" package3d_urn="urn:adsk.eagle:package:15796/2" value="BLUE"/>
+<part name="LED2" library="led" library_urn="urn:adsk.eagle:library:259" deviceset="LED" device="SMT1206" package3d_urn="urn:adsk.eagle:package:15796/2" value="RED"/>
+<part name="LED3" library="led" library_urn="urn:adsk.eagle:library:259" deviceset="LED" device="SMT1206" package3d_urn="urn:adsk.eagle:package:15796/2" value="YELLOW"/>
 <part name="P+10" library="supply1" library_urn="urn:adsk.eagle:library:371" deviceset="+15V" device=""/>
-<part name="R19" library="rcl" library_urn="urn:adsk.eagle:library:334" deviceset="R-US_" device="R0603" package3d_urn="urn:adsk.eagle:package:23555/3" value="1k"/>
+<part name="R19" library="rcl" library_urn="urn:adsk.eagle:library:334" deviceset="R-US_" device="R0603" package3d_urn="urn:adsk.eagle:package:23555/3" value="100k"/>
 <part name="GND23" library="supply1" library_urn="urn:adsk.eagle:library:371" deviceset="GND" device=""/>
 <part name="+3V10" library="supply1" library_urn="urn:adsk.eagle:library:371" deviceset="+3V3" device=""/>
@@
 <part name="GND24" library="supply1" library_urn="urn:adsk.eagle:library:371" deviceset="GND" device=""/>
 <part name="P-8" library="supply1" library_urn="urn:adsk.eagle:library:371" deviceset="-15V" device=""/>
-<part name="R21" library="rcl" library_urn="urn:adsk.eagle:library:334" deviceset="R-US_" device="R0603" package3d_urn="urn:adsk.eagle:package:23555/3" value="1k"/>
+<part name="R21" library="rcl" library_urn="urn:adsk.eagle:library:334" deviceset="R-US_" device="R0603" package3d_urn="urn:adsk.eagle:package:23555/3" value="10k"/>
 <part name="GND25" library="supply1" library_urn="urn:adsk.eagle:library:371" deviceset="GND" device=""/>
-<part name="LED4" library="led" library_urn="urn:adsk.eagle:library:259" deviceset="LED" device="SMT1206" package3d_urn="urn:adsk.eagle:package:15796/2"/>
-<part name="R22" library="rcl" library_urn="urn:adsk.eagle:library:334" deviceset="R-US_" device="R0603" package3d_urn="urn:adsk.eagle:package:23555/3" value="1k"/>
+<part name="LED4" library="led" library_urn="urn:adsk.eagle:library:259" deviceset="LED" device="SMT1206" package3d_urn="urn:adsk.eagle:package:15796/2" value="GREEN"/>
+<part name="R22" library="rcl" library_urn="urn:adsk.eagle:library:334" deviceset="R-US_" device="R0603" package3d_urn="urn:adsk.eagle:package:23555/3" value="470R"/>
 <part name="GND26" library="supply1" library_urn="urn:adsk.eagle:library:371" deviceset="GND" device=""/>
 <part name="U$6" library="synth" deviceset="SWITCH-DPDT" device=""/>

Commit message: Found error in sch values around lin->exp converter
Parts:
- added R23, R24: 1k, rcl:R-US_R0603
- C20: value 10u -> 10p
- Q1, Q2: SPICEPREFIX (none) -> Q
- R9: value 2.7M -> 845k
- SJ1: SPICEPREFIX (none) -> B
- U$11: SPICEPREFIX (none) -> U
Connections:
- new net N$23: Q2B.E, R23.1
- new net N$24: Q2A.E, R24.1
- net +15V: now also R23.2, R24.2; no longer Q2A.E, Q2B.E
Other:
- moved on the sheet: C20, Q1A, Q1B, Q2A, Q2B, R8, R9, SJ1

Commit message: Changed board rails, transferred sims to pcb
Parts:
- removed TP5: TPPAD1-13, testpad:TPPAD1-13
- removed U$10: (no value), LITTLEBITS:XX-13700DMP16
- removed U$11, U$5: TL072, synth:TL072
- removed U$2: STM32C8, synth:STM32C8
- added C27: 2000p, rcl:C-EUC0603
- added C28: 1000p, rcl:C-EUC0603
- added C29, C30, C31, C32, C33, C34: 0.1u, rcl:C-EUC0603
- added D1, D2, D3, D4, D5, D6: 1N4148, LITTLEBITS:DIODESOD123
- added Q3: (no value), LITTLEBITS:TRANS-BJT_NPN-DUAL-BC847BS-JBLMASK
- added Q4: (no value), LITTLEBITS:TRANS-BJT_PNP-DUAL-BC857-JBLMASK
- added R25, R45: 30k, rcl:R-US_R0603
- added R28: 562k, rcl:R-US_R0603
- added R37, R43, R44: 10k, rcl:R-US_R0603
- added R38: 3.3k, rcl:R-US_R0603
- added R39: 100k, rcl:R-US_R0603
- added R40: 14.7k, rcl:R-US_R0603
- added R41: 1.6k, rcl:R-US_R0603
- added R42: 8.45k, rcl:R-US_R0603
- added R46: 10, rcl:R-US_R0603
- added SJ2: (no value), jumper:SJ
- added TP1, TP2: TPPAD1-13, testpad:TPPAD1-13
- added U11, U12, U4, U5, U7, U9: TL072, synth:TL072
- added U6, U8: (no value), LITTLEBITS:XX-13700DMP16
- added VR1, VR2: 1k, LITTLEBITS:POT-TRIM-SMD-BOURNS-3314J-1
- C1: value 0.1u -> 10p
- C3: value 0.1u -> 1000p
- C4: value 22p -> 2000p
- C42: value 1000p -> 2200p
- C43: value 2000p -> 2200p
- C7: value 1000p -> 0.1u
- C8: value 2000p -> 0.1u
- R1: value 22k -> 3.5k
- R10: value 20k -> 10k
- R13: value 330k -> 165k
- R14: value 5.1k -> 1k
- R15: value 20k -> 570
- R16: value 330k -> 72k
- R17: value 4.7k -> 570
- R18: value 4.7k -> 72k
- R2: value 22k -> 30k
- R23, R24: value 1k -> 10
- R26, R33, R35: value 100k -> 10k
- R27, R30, R32, R34: value 2k -> 220
- R29: value 100K -> 10k
- R3: value 4.7k -> 10k
- R31: value 10k -> 10
- R36: value 10k -> 3.3k
- R4: value 1k -> 10k
- R6: value 10k -> 165k
- R9: value 845k -> 280k
- U$1: value TL072 -> TRS; device synth:TL072 -> synth:TRS
- U1: value THAT2180 -> STM32C8; device synth:THAT2180 -> synth:STM32C8
- renumbered U$3 to U2, U$4 to U3
Connections:
- removed net N$3: C4.1, R2.1, U$1G$1.IN-, U1.OUT
- removed net VCA_OUT0: C4.2, R2.2, TP4.TP, U$1G$1.OUT
- new net N$25: C43.1, U6G$2.OUT, U7G$2.IN+
- new net N$26: R36.2, U8G$1.OUT, U9G$2.IN+
- new net N$28: C42.1, U6G$1.OUT, U7G$1.IN+
- new net N$29: R25.1, U8G$1.+IN, VR1.3
- new net N$30: U8G$1.-IN, VR1.1
- new net N$37: D2.C, D3.A
- new net N$38: D1.C, D2.A
- new net N$39: D4.C, D5.A
- new net N$40: D5.C, D6.A
- new net N$41: R40.1, R41.2, R42.1
- new net N$42: R39.1, R40.2, U5G$1.IN-
- new net N$43: R39.2, R43.1, U5G$1.OUT
- new net N$44: C27.1, R43.2, R44.1
- new net N$45: C28.1, R44.2, U5G$2.IN+
- new net N$46: R45.1, U8G$1.AMP/BIAS
- new net N$47: U8G$2.-IN, VR2.1
- new net N$48: C1.1, Q3A.C, R28.1, U11G$2.IN-
- new net N$49: R29.2, R33.1, U7G$1.IN-, U7G$1.OUT
- new net N$50: R17.1, R18.2, U12G$2.IN+
- new net N$51: Q3B.C, Q4A.B, Q4B.B, Q4B.C
- new net N$52: Q4A.C, SJ2.2
- new net N$53: Q4B.E, R31.1
- new net N$54: Q4A.E, R46.1
- new net Q-CTRL0-I: C27.2, R45.2, U5G$2.IN-, U5G$2.OUT
- new net VCA-OUT0: R1.1, TP4.TP, U$1.T, U11G$1.OUT
- new net VCA0-EXP: SJ2.1, U8G$2.AMP/BIAS
- net +15V: now also C29.1, C31.2, C33.1, C8.2, R16.1, R18.1, R28.2, R31.2, R42.2, R46.2, U11G$3.V+, U12G$3.V+, U4G$3.V+, U5G$3.V+, U6G$3.VCC, U7G$3.V+, U8G$3.VCC, U9G$3.V+; no longer C3.2, U$10G$3.VCC, U$11G$3.V+, U$1G$3.V+, U$5G$3.V+, U1.V+
- net +3V3: now also U1.VDD@1, U1.VDD@2, U1.VDDA; no longer R18.2, U$2.VDD@1, U$2.VDD@2, U$2.VDDA
- net -15V: now also C28.2, C3.2, C30.2, C32.1, C34.2, U11G$3.V-, U12G$3.V-, U4G$3.V-, U5G$3.V-, U6G$3.GND, U7G$3.V-, U8G$3.GND, U9G$3.V-; no longer C1.1, R14.1, R31.2, R36.2, U$10G$3.GND, U$11G$3.V-, U$1G$3.V-, U$5G$3.V-
- net F-CTRL0: now also R6.2, U1.PA9; no longer U$2.PA9
- net F-CTRL0-EXP: now also U6G$1.AMP/BIAS, U6G$2.AMP/BIAS; no longer U$10G$1.AMP/BIAS, U$10G$2.AMP/BIAS
- net F-CTRL0-LIN: now also U4G$1.IN-, U4G$1.OUT; no longer U$11G$2.IN-, U$11G$2.OUT
- net F-CTRL1: now also U1.PA0; no longer U$2.PA0
- net F-CTRL2: now also U1.PA3; no longer U$2.PA3
- net F-CTRL3: now also U1.PB0; no longer U$2.PB0
- net F0-OUT: now also R2.1, R2.2, R25.2, R35.2, U7G$2.IN-, U7G$2.OUT, U8G$2.+IN, VR2.3; no longer C42.2, R1.1, R35.1, R36.1, U$10G$2.BUFF/OUT
- net GND: now also C29.2, C30.1, C31.1, C32.2, C33.2, C34.1, C7.2, C8.1, Q3B.B, R17.2, R36.1, R38.1, R41.1, U$1.S, U1.VSS@1, U1.VSS@2, U1.VSSA, U11G$1.IN+, U11G$2.IN+, U9G$1.IN+, VR1.2, VR2.2; no longer C1.2, C3.1, R17.1, R4.1, U$11G$1.IN+, U$1G$1.IN+, U$2.VSS@1, U$2.VSS@2, U$2.VSSA, U1.EC+, U1.GND
- net LED: now also U1.PA15; no longer U$2.PA15
- net MOSI: now also U1.PA7; no longer U$2.PA7
- net N$1: now also U4G$2.IN-; no longer U$5G$2.IN-
- net N$10: now also U9G$1.OUT; no longer U$11G$1.OUT
- net N$11: now also U9G$1.IN-; no longer U$11G$1.IN-
- net N$12: now also U4G$1.IN+; no longer U$11G$2.IN+
- net N$15: now also U4G$2.OUT; no longer U$5G$2.OUT
- net N$16: now also Q3A.E, Q3B.E; no longer U1.V-
- net N$19: now also R5.2, R6.1, U12G$2.IN-; no longer R16.1, R17.2, R18.1
- net N$2: now also U11G$1.IN-, U8G$2.OUT; no longer U1.-IN
- net N$20: now also U4G$2.IN+; no longer U$5G$2.IN+
- net N$27: now also U6G$1.+IN; no longer U$10G$1.+IN
- net N$31: now also R29.1, U6G$1.-IN; no longer R29.2, U$10G$1.-IN
- net N$32: now also D1.A, D6.C, R37.1, R38.2, U9G$2.IN-; no longer C42.1, U$10G$1.BUFF/IN, U$10G$1.OUT
- net N$33: now also C1.2, R14.1, U11G$2.OUT; no longer R29.1, R31.1, R33.1, U$10G$1.BUFF/OUT
- net N$34: now also C42.2, D3.C, D4.A, R37.2, U9G$2.OUT; no longer C43.1, U$10G$2.BUFF/IN, U$10G$2.OUT
- net N$35: now also U6G$2.+IN; no longer U$10G$2.+IN
- net N$36: now also R35.1, U6G$2.-IN; no longer R35.2, U$10G$2.-IN
- net N$4: now also C3.1, U12G$1.IN+; no longer R4.2, R5.2
- net N$5: now also C4.1, R3.1, R4.2; no longer C8.2, R5.1, R6.2
- net N$6: now also R4.1, R5.1, TP2.TP, U12G$2.OUT; no longer C7.2, R6.1, U$1G$2.IN+
- net N$8: now also U1.BOOT0; no longer U$2.BOOT0
- net NRST: now also U1.NRST; no longer U$2.NRST
- net NSS: now also U1.PA4; no longer U$2.PA4
- net Q-CTRL0: now also U1.PA10, U5G$1.IN+; no longer U$2.PA10
- net Q-CTRL1: now also U1.PA1; no longer U$2.PA1
- net Q-CTRL2: now also U1.PB4; no longer U$2.PB4
- net Q-CTRL3: now also U1.PB1; no longer U$2.PB1
- net SCK: now also U1.PA5; no longer U$2.PA5
- net SWCLK: now also U1.PA14; no longer U$2.PA14
- net SWDIO: now also U1.PA13; no longer U$2.PA13
- net SWO: now also U1.PB3; no longer U$2.PB3
- net VCA-CTRL0: now also U1.PA8; no longer R3.1, U$2.PA8
- net VCA-CTRL1: now also U1.PA11; no longer U$2.PA11
- net VCA-CTRL2: now also U1.PA2; no longer U$2.PA2
- net VCA-CTRL3: now also U1.PB5; no longer U$2.PB5
- net VCA0-LP: now also C4.2, Q3A.B, TP1.TP, U12G$1.IN-, U12G$1.OUT; no longer C8.1, TP5.TP, U$1G$2.IN-, U$1G$2.OUT, U1.EC-

Commit message: Standardize part vals
Parts:
- removed TP8: TPPAD1-13, testpad:TPPAD1-13
- removed U$1: TRS, synth:TRS
- added JP2: (no value), pinhead:PINHD-1X3
- added TP5: TPPAD1-13, testpad:TPPAD1-13
- C35, C36: value 2200p -> 2000p
- C9: value .01u -> 0.01u
- JP7: value (none) -> TRS; device pinhead:PINHD-1X3 -> synth:TRS
- Q1, Q3: value (none) -> BC847BS
- Q2, Q4: value (none) -> BC857BS
- R1: value 3.5k -> 3.48k
- R15, R17: value 570 -> 562
- R41: value 1.6k -> 1.62k
- U6, U8: value (none) -> LM13700
- renumbered C42 to C35, C43 to C36, C44 to C37, C45 to C38, JP10 to JP5, JP11 to JP6, JP8 to JP3, JP9 to JP4, U$6 to SW1, U12 to U10
Connections:
- net +15V renamed +12V
- net -15V renamed -12V
- new net N$3: R2.2, U8G$2.+IN, VR2.3
- net -15V-IN: now also JP2.1; no longer JP7.1
- net 15V-IN: now also JP2.3; no longer JP7.3
- net F-CTRL0-LIN: now also TP6.TP; no longer TP7.TP
- net F0-OUT: now also TP5.TP; no longer R2.2, TP6.TP, U8G$2.+IN, VR2.3
- net GND: now also JP2.2, JP7.S; no longer JP7.2, U$1.S
- net N$15: now also TP7.TP; no longer TP8.TP
- net VCA-OUT0: now also JP7.T; no longer U$1.T
Other:
- moved on the sheet: TP6, TP7
