File: pcb/1-voice/3_3/1-voice(3_3).brd (EAGLE design)
At the start: 72.6 x 30 mm, 128 parts, among them Q1 BC847BS, Q2 BC857BS, Q3 BC847BS, Q4 BC857BS, SW1 SWITCH-DPDT, U1 STM32C8, U10 TL072, U11 TL072, U2 DAC084S085, U3 TLV760, U4 TL072, U5 TL072, U6 LM13700, U7 TL072, U8 LM13700, U9 TL072

Commit message: Finished latest layout
Parts:
- removed C10, C21, C22: 1u, rcl:C0603
- removed C11, C12, C14, C16: 0.1u, rcl:C0603
- removed C13: 4.7u, rcl:C0603
- removed C15, C17: 10u, rcl:C0603
- removed C9: 0.01u, rcl:C0603
- removed JP1: (no value), pinhead:1X06
- removed JP3, JP4, JP5, JP6: (no value), pinhead:1X04
- removed LED2: RED, led:1206
- removed LED4: GREEN, led:1206
- removed R20: 1k, rcl:R0603
- removed R22: 470R, rcl:R0603
- removed R7: 10k, rcl:R0603
- removed SJ1, SJ2: (no value), jumper:SJ
- removed TP1, TP2, TP3, TP4, TP5, TP6, TP7: TPPAD1-13, testpad:P1-13
- removed U1: STM32C8, synth:LQFP48
- removed U2: DAC084S085, synth:VSSOP10
- removed U3: TLV760, synth:SOT23-3
- added U$1: CV_MODULE, synth:CV_MODULE
- added U$2, U$3: CURRENT_TESTPOINT, synth:CURRENT_TESTPOINT
- D1, D2, D3, D4, D5, D6: device LITTLEBITS:SOD123 -> LITTLEBITS:SOD-323
- R1: value 3.48k -> 3.3k
- moved JP7 237.6 mm to (91.4, 5.70), turned to 180 degrees
- moved C8 220.6 mm to (37.5, 19.8)
- moved R5 210.3 mm to (34.3, 19.8), turned to 180 degrees
- moved C7 207.9 mm to (34.3, 12.4), turned to 180 degrees
- moved R4 203.5 mm to (41.4, 18.2)
- moved R2 201.2 mm to (87.9, 24.5)
- moved R3 200.9 mm to (41.4, 14.0), turned to 180 degrees
- moved C4 199.9 mm to (41.4, 16.1), turned to 180 degrees
- moved R18 198.9 mm to (30.4, 14.0), turned to 180 degrees
- moved R6 196.3 mm to (30.4, 18.2), turned to 180 degrees
- moved R17 192.9 mm to (30.4, 16.1), turned to 180 degrees
- moved U10 191.9 mm to (35.9, 16.1), turned to 270 degrees
- moved R1 189.8 mm to (85.8, 16.7), turned to 270 degrees
- moved C3 186.7 mm to (37.5, 12.4), turned to 180 degrees
- moved Q3 183.5 mm to (49.0, 5.80), turned to 180 degrees
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Connections:
- removed net +3V3: C10.1, C11.1, C12.1, C13.1, C14.1, C15.1, C16.1, C17.1, C22.1, C9.1, JP1.5, LED2.A, TP3.TP, U1.P$24, U1.P$48, U1.P$9, U2.P$1, U2.P$7, U3.P$1
- removed net -15V-IN: JP2.1, SW1.P$5
- removed net 15V-IN: JP2.3, SW1.P$2
- removed net F-CTRL1: JP6.3, U1.P$10
- removed net F-CTRL2: JP3.3, U1.P$13
- removed net F-CTRL3: JP4.3, U1.P$18
- removed net LED: LED4.A, U1.P$38
- removed net MOSI: U1.P$17, U2.P$8
- removed net N$18: LED2.C, R20.2
- removed net N$22: LED4.C, R22.2
- removed net N$26: R36.2, U8.5, U9.P$5
- removed net N$52: Q4.6, SJ2.2
- removed net NRST: JP1.2, U1.P$7
- removed net NSS: U1.P$14, U2.P$9
- removed net OSC1-OUT: JP6.1, U2.P$3
- removed net OSC2-OUT: JP3.1, U2.P$4
- removed net OSC3-OUT: JP4.1, U2.P$5
- removed net Q-CTRL1: JP6.4, U1.P$11
- removed net Q-CTRL2: JP3.4, U1.P$40
- removed net Q-CTRL3: JP4.4, U1.P$19
- removed net SCK: U1.P$15, U2.P$10
- removed net SWCLK: JP1.3, U1.P$37
- removed net SWDIO: JP1.4, U1.P$34
- removed net SWO: JP1.1, U1.P$39
- removed net VCA-CTRL1: JP6.2, U1.P$32
- removed net VCA-CTRL2: JP3.2, U1.P$12
- removed net VCA-CTRL3: JP4.2, U1.P$41
- new net -12V-IN: JP2.1, SW1.P$2
- new net 12V-IN: JP2.3, SW1.P$5
- new net N$55: R25.1, U8.3, VR1.3
- net +12V: now also SW1.P$4, U$1.VCC; no longer C21.1, SW1.P$1, U3.P$2
- net -12V: now also SW1.P$1; no longer SW1.P$4
- net F-CTRL0: now also U$1.CV1-4; no longer JP5.3, R6.2, U1.P$30
- net F-CTRL0-EXP: now also U$2.P1, U$2.P1.1; no longer SJ1.1
- net F-CTRL0-LIN: now also U4.P$6, U4.P$7; no longer TP6.TP, U4.P$1, U4.P$2
- net F0-OUT: no longer TP5.TP
- net GND: now also Q3.2, U$1.GND, U9.P$5; no longer C10.2, C11.2, C12.2, C13.2, C14.2, C15.2, C16.2, C17.2, C21.2, C22.2, C9.2, JP1.6, Q3.5, R20.1, R22.1, R7.2, U1.P$23, U1.P$47, U1.P$8, U11.P$3, U2.P$6, U3.P$3
- net N$1: now also U4.P$2; no longer U4.P$6
- net N$12: now also U4.P$5; no longer U4.P$3
- net N$15: now also U4.P$1; no longer TP7.TP, U4.P$7
- net N$19: now also U10.P$2; no longer U10.P$6
- net N$2: now also U11.P$6; no longer U11.P$2
- net N$20: now also U4.P$3; no longer U4.P$5
- net N$29: now also R36.2, U11.P$3, U8.5; no longer R25.1, U8.3, VR1.1
- net N$30: now also VR1.1; no longer VR1.3
- net N$32: now also D1.2, D6.1, U11.P$2; no longer D1.A, D6.C, U9.P$6
- net N$33: now also U9.P$7; no longer U11.P$7
- net N$34: now also D3.1, D4.2, U11.P$1; no longer D3.C, D4.A, U9.P$7
- net N$37: now also D2.1, D3.2; no longer D2.C, D3.A
- net N$38: now also D1.1, D2.2; no longer D1.C, D2.A
- net N$39: now also D4.1, D5.2; no longer D4.C, D5.A
- net N$4: now also U10.P$5; no longer U10.P$3
- net N$40: now also D5.1, D6.2; no longer D5.C, D6.A
- net N$48: now also Q3.3, U9.P$6; no longer Q3.6, U11.P$6
- net N$50: now also U10.P$3; no longer U10.P$5
- net N$51: now also Q3.6; no longer Q3.3
- net N$6: now also U10.P$1; no longer TP2.TP, U10.P$7
- net N$7: now also U$2.P2, U$2.P2.1; no longer SJ1.2
- net N$8: now also Q4.6, U$3.P2, U$3.P2.1; no longer R7.1, U1.P$44
- net OSC0-OUT: now also U$1.OSC-4; no longer JP5.1, U2.P$2
- net Q-CTRL0: now also U$1.CV3-4; no longer JP5.4, U1.P$31
- net VCA-CTRL0: now also R6.2, U$1.CV2-4; no longer JP5.2, U1.P$29
- net VCA-OUT0: now also U11.P$7; no longer TP4.TP, U11.P$1
- net VCA0-EXP: now also U$3.P1, U$3.P1.1; no longer SJ2.1
- net VCA0-LP: now also Q3.5, U10.P$6, U10.P$7; no longer Q3.2, TP1.TP, U10.P$1, U10.P$2
Routing:
- net +12V: track 120.5 -> 262.3 mm, vias 10 -> 23
- net +3V3: track 102.6 -> 0.00 mm, vias 3 -> 0
- net VCA-CTRL0: track 81.7 -> 5.83 mm, vias 4 -> 0
- net N$46: track 0.00 -> 70.6 mm, vias 0 -> 2
- net -12V: track 155.2 -> 221.9 mm, vias 9 -> 10
- net VCA0-EXP: track 0.00 -> 59.0 mm, vias 0 -> 1
- net F0-OUT: track 2.63 -> 58.7 mm, vias 0 -> 5
- net F-CTRL0: track 47.0 -> 10.9 mm, vias 3 -> 0
- net Q-CTRL2: track 28.8 -> 0.00 mm, vias 1 -> 0
- net VCA-CTRL1: track 25.6 -> 0.00 mm, vias 1 -> 0
- net F-CTRL1: track 25.0 -> 0.00 mm, vias 1 -> 0
- net VCA0-LP: track 0.00 -> 24.7 mm, vias 0 -> 4
- net VCA-CTRL3: track 24.6 -> 0.00 mm, vias 1 -> 0
- net N$32: track 0.00 -> 23.4 mm, vias 0 -> 2
- net Q-CTRL1: track 22.3 -> 0.00 mm, vias 1 -> 0
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Other:
- board size 72.6 x 30 mm -> 92.6 x 37.1 mm
- board text added: "190719"
- board text added: "F-CTRL"
- board text added: "Low-pass Filter"
- board text added: "VCA-CTRL"
- board text removed: "+15V"
- board text removed: "-15V"
- board text removed: "1-Voice "Synth""
- board text removed: "190521"
- board text removed: "3V3"
- board text removed: "F"
- board text removed: "F In"
- board text removed: "F Lin"
- board text removed: "Filtered"
- board text removed: "GND"
- board text removed: "Osc"
- board text removed: "Q"
- board text removed: "VCA"
- board text removed: "VCA LP"
- board text removed: "VCA OUT"
- board text removed: "Voice 0"
- board text removed: "Voice 1"
- board text removed: "Voice 2"
