File: pcb/digital-interface/1_1/digital_interface(1_1).sch (EAGLE design)
At the start: 98 parts, among them Q1 BC847BS, Q2 BC857BS, Q3 BC847BS, Q4 BC857BS, SW1 SWITCH-DPDT, U10 TL072, U11 TL072, U4 TL072, U5 TL072, U6 LM13700, U7 TL072, U8 LM13700, U9 TL072

Commit message: Finished latest layout
Parts:
- removed C1, C20: 10p, rcl:C-EUC0603
- removed C18, C19, C25, C26, C29, C30, C31, C32, C33, C34, C37, C38, C5, C6, C7, C8: 0.1u, rcl:C-EUC0603
- removed C2: 10u, rcl:C-EUC0603
- removed C23, C28, C3: 1000p, rcl:C-EUC0603
- removed C24, C27, C35, C36, C4: 2000p, rcl:C-EUC0603
- removed D1, D2, D3, D4, D5, D6: 1N4148, LITTLEBITS:DIODESOD
- removed JP2: (no value), pinhead:PINHD-1X3
- removed JP7: TRS, synth:TRS
- removed LED1: BLUE, led:LEDSMT1206
- removed LED3: YELLOW, led:LEDSMT1206
- removed Q1, Q3: BC847BS, LITTLEBITS:TRANS-BJT_NPN-DUAL-BC847BS-JBLMASK
- removed Q2, Q4: BC857BS, LITTLEBITS:TRANS-BJT_PNP-DUAL-BC857-JBLMASK
- removed R1, R36, R38: 3.3k, rcl:R-US_R0603
- removed R10, R11, R12, R21, R26, R29, R3, R33, R35, R37, R4, R43, R44, R5: 10k, rcl:R-US_R0603
- removed R13, R6: 165k, rcl:R-US_R0603
- removed R14, R8: 1k, rcl:R-US_R0603
- removed R15, R17: 562, rcl:R-US_R0603
- removed R16, R18: 72k, rcl:R-US_R0603
- removed R19, R39: 100k, rcl:R-US_R0603
- removed R2, R25, R45: 30k, rcl:R-US_R0603
- removed R23, R24, R31, R46: 10, rcl:R-US_R0603
- removed R27, R30, R32, R34: 220, rcl:R-US_R0603
- removed R28: 562k, rcl:R-US_R0603
- removed R40: 14.7k, rcl:R-US_R0603
- removed R41: 1.62k, rcl:R-US_R0603
- removed R42: 8.45k, rcl:R-US_R0603
- removed R9: 280k, rcl:R-US_R0603
- removed SW1: SWITCH-DPDT, synth:SWITCH-DPDT
- removed U$2, U$3: CURRENT_TESTPOINT, synth:CURRENT_TESTPOINT
- removed U10, U11, U4, U5, U7, U9: TL072, synth:TL072
- removed U6, U8: LM13700, LITTLEBITS:XX-13700DMP16
- removed VR1, VR2: 1k, LITTLEBITS:POT-TRIM-SMD-BOURNS-3314J-1
- added C10, C21, C22: 1u, rcl:C-EUC0603
- added C11, C12, C14, C16: 0.1u, rcl:C-EUC0603
- added C13: 4.7u, rcl:C-EUC0603
- added C15, C17: 10u, rcl:C-EUC0603
- added C9: 0.01u, rcl:C-EUC0603
- added JP1: (no value), pinhead:PINHD-1X6
- added LED2: RED, led:LEDSMT1206
- added LED4: GREEN, led:LEDSMT1206
- added R20: 1k, rcl:R-US_R0603
- added R22: 470R, rcl:R-US_R0603
- added R7: 10k, rcl:R-US_R0603
- added U1: STM32C8, synth:STM32C8
- added U2: DAC084S085, synth:DAC084S085
- added U3: TLV760, synth:TLV760
Connections:
- removed net -12V: C19.1, C23.2, C26.1, C28.2, C3.2, C30.2, C32.1, C34.2, C38.2, C6.1, C7.1, LED3.C, SW1.P$1, U10G$3.V-, U11G$3.V-, U4G$3.V-, U5G$3.V-, U6G$3.GND, U7G$3.V-, U8G$3.GND, U9G$3.V-
- removed net -12V-IN: JP2.1, SW1.P$2
- removed net 12V-IN: JP2.3, SW1.P$5
- removed net F-CTRL0-EXP: U$2.P1, U6G$1.AMP/BIAS, U6G$2.AMP/BIAS
- removed net F-CTRL0-LIN: C24.2, Q1A.B, U4G$2.IN-, U4G$2.OUT
- removed net F0-OUT: R2.1, R25.2, R35.2, U7G$2.IN-, U7G$2.OUT
- removed net FILT_IN: C2.2, R26.1
- removed net N$1: R10.2, R13.1, U4G$1.IN-
- removed net N$10: C20.2, R8.1, U9G$1.OUT
- removed net N$11: C20.1, Q1A.C, R9.1, U9G$1.IN-
- removed net N$12: C23.1, R11.2, U4G$2.IN+
- removed net N$13: Q1B.C, Q2A.B, Q2B.B, Q2B.C
- removed net N$14: C24.1, R11.1, R12.2
- removed net N$15: R10.1, R12.1, U4G$1.OUT
- removed net N$16: Q3A.E, Q3B.E, R14.2
- removed net N$17: LED1.C, R19.2
- removed net N$19: R5.2, R6.1, U10G$1.IN-
- removed net N$2: R1.2, U11G$2.IN-, U8G$2.OUT
- removed net N$20: R15.1, R16.2, U4G$1.IN+
- removed net N$21: LED3.A, R21.2
- removed net N$23: Q2B.E, R23.1
- removed net N$24: Q2A.E, R24.1
- removed net N$25: C36.1, U6G$2.OUT, U7G$2.IN+
- removed net N$27: R26.2, R27.2, U6G$1.+IN
- removed net N$28: C35.1, U6G$1.OUT, U7G$1.IN+
- removed net N$29: R36.2, U11G$1.IN+, U8G$1.OUT
- removed net N$3: R2.2, U8G$2.+IN, VR2.3
- removed net N$30: U8G$1.-IN, VR1.3
- removed net N$31: R29.1, R30.1, U6G$1.-IN
- removed net N$32: D1.A, D6.C, R37.1, R38.2, U11G$1.IN-
- removed net N$33: C1.2, R14.1, U9G$2.OUT
- removed net N$34: C35.2, D3.C, D4.A, R37.2, U11G$1.OUT
- removed net N$35: R32.1, R33.2, U6G$2.+IN
- removed net N$36: R34.1, R35.1, U6G$2.-IN
- removed net N$37: D2.C, D3.A
- removed net N$38: D1.C, D2.A
- removed net N$39: D4.C, D5.A
- removed net N$4: C3.1, R3.2, U10G$2.IN+
- removed net N$40: D5.C, D6.A
- removed net N$41: R40.1, R41.2, R42.1
- removed net N$42: R39.1, R40.2, U5G$1.IN-
- removed net N$43: R39.2, R43.1, U5G$1.OUT
- removed net N$44: C27.1, R43.2, R44.1
- removed net N$45: C28.1, R44.2, U5G$2.IN+
- removed net N$46: R45.1, U8G$1.AMP/BIAS
- removed net N$47: U8G$2.-IN, VR2.1
- removed net N$48: C1.1, Q3B.C, R28.1, U9G$2.IN-
- removed net N$49: R29.2, R33.1, U7G$1.IN-, U7G$1.OUT
- removed net N$5: C4.1, R3.1, R4.2
- removed net N$50: R17.1, R18.2, U10G$1.IN+
- removed net N$51: Q3A.C, Q4A.B, Q4B.B, Q4B.C
- removed net N$53: Q4B.E, R31.1
- removed net N$54: Q4A.E, R46.1
- removed net N$55: R25.1, U8G$1.+IN, VR1.1
- removed net N$6: R4.1, R5.1, U10G$1.OUT
- removed net N$7: Q2A.C, U$2.P2
- removed net N$9: Q1A.E, Q1B.E, R8.2
- removed net Q-CTRL0-I: C27.2, R45.2, U5G$2.IN-, U5G$2.OUT
- removed net VCA-OUT0: JP7.T, R1.1, U11G$2.OUT
- removed net VCA0-EXP: U$3.P1, U8G$2.AMP/BIAS
- removed net VCA0-LP: C4.2, Q3B.B, U10G$2.IN-, U10G$2.OUT
- new net +3V3: C10.1, C11.1, C12.1, C13.1, C14.1, C15.1, C16.1, C17.1, C22.1, C9.1, JP1.5, LED2.A, U1.VDD@1, U1.VDD@2, U1.VDDA, U2.VA, U2.V_REFIN, U3.VOUT
- new net F-CTRL1: U$1.CV2-1, U1.PA0
- new net F-CTRL2: U$1.CV2-3, U1.PA3
- new net F-CTRL3: U$1.CV2-4, U1.PB0
- new net LED: LED4.A, U1.PA15
- new net MOSI: U1.PA7, U2.DIN
- new net N$18: LED2.C, R20.2
- new net N$22: LED4.C, R22.2
- new net NRST: JP1.4, U1.NRST
- new net NSS: U1.PA4, U2.!SYNC
- new net OSC1-OUT: U$1.OSC-1, U2.V_OUTB
- new net OSC2-OUT: U$1.OSC-3, U2.V_OUTC
- new net OSC3-OUT: U$1.OSC-4, U2.V_OUTD
- new net Q-CTRL1: U$1.CV3-1, U1.PA1
- new net Q-CTRL2: U$1.CV3-3, U1.PB4
- new net Q-CTRL3: U$1.CV3-4, U1.PB1
- new net SCK: U1.PA5, U2.SCLK
- new net SWCLK: JP1.2, U1.PA14
- new net SWDIO: JP1.3, U1.PA13
- new net SWO: JP1.1, U1.PB3
- new net VCA-CTRL1: U$1.CV1-1, U1.PA11
- new net VCA-CTRL2: U$1.CV1-3, U1.PA2
- new net VCA-CTRL3: U$1.CV1-4, U1.PB5
- net +12V: now also C21.1, U3.VIN; no longer C18.2, C25.2, C29.1, C31.2, C33.1, C37.1, C5.2, C8.2, LED1.A, R16.1, R18.1, R23.2, R24.2, R28.2, R31.2, R42.2, R46.2, R9.2, SW1.P$4, U10G$3.V+, U11G$3.V+, U4G$3.V+, U5G$3.V+, U6G$3.VCC, U7G$3.V+, U8G$3.VCC, U9G$3.V+
- net F-CTRL0: now also U$1.CV2-2, U1.PA9; no longer R13.2, U$1.CV1-4
- net GND: now also C10.2, C11.2, C12.2, C13.2, C14.2, C15.2, C16.2, C17.2, C21.2, C22.2, C9.2, JP1.6, R20.1, R22.1, R7.2, U1.VSS@1, U1.VSS@2, U1.VSSA, U2.GND, U3.GND; no longer C18.1, C19.2, C25.1, C26.2, C29.2, C30.1, C31.1, C32.2, C33.2, C34.1, C36.2, C37.2, C38.1, C5.1, C6.2, C7.2, C8.1, JP2.2, JP7.S, Q1B.B, Q3A.B, R15.2, R17.2, R19.1, R21.1, R27.1, R30.2, R32.2, R34.2, R36.1, R38.1, R41.1, U11G$2.IN+, U9G$1.IN+, U9G$2.IN+, VR1.2, VR2.2
- net N$8: now also R7.1, U1.BOOT0; no longer Q4A.C, U$3.P2
- net OSC0-OUT: now also U$1.OSC-2, U2.V_OUTA; no longer C2.1, U$1.OSC-4
- net Q-CTRL0: now also U$1.CV3-2, U1.PA10; no longer U$1.CV3-4, U5G$1.IN+
- net VCA-CTRL0: now also U$1.CV1-2, U1.PA8; no longer R6.2, U$1.CV2-4
Other:
- note added: "VDD VSS"
- note added: "VDDA VSSA"
